Commit message: update the static walk controller

File: quadruped_model/urdf/quadruped_model.urdf (robot description, URDF)
Before this commit: robot quadruped_model, 17 links, 16 joints
Links:
- added link world, mass 27.801
Joints:
- added joint fixed_1_joint: type revolute, parent world, child base_link, origin xyz=0.427 0.075 -0.0095 rpy=0 1.5708 0, axis 0 0 1, limit lower=-3.0 upper=3.0 effort=300 velocity=10
